Commit message: Added open and closed poses

File: config/panda_arm_hand.srdf.xacro (robot description, xacro)
@@ -28,4 +28,12 @@
     <joint name="panda_joint7" value="0.785" />
   </group_state>
+  <group_state name="open" group="hand">
+    <joint name="panda_finger_joint1" value="0.035" />
+    <joint name="panda_finger_joint2" value="0.035" />
+  </group_state>
+  <group_state name="closed" group="hand">
+    <joint name="panda_finger_joint1" value="0" />
+    <joint name="panda_finger_joint2" value="0" />
+  </group_state>
   <!--END EFFECTOR: Purpose: Represent information about an end effector.-->
   <end_effector name="hand" parent_link="panda_link8" group="hand" parent_group="panda_arm" />

Commit message: Added open and closed poses (#34)

File: config/panda_arm_hand.srdf.xacro (robot description, xacro)
@@ -28,4 +28,12 @@
     <joint name="panda_joint7" value="0.785" />
   </group_state>
+  <group_state name="open" group="hand">
+    <joint name="panda_finger_joint1" value="0.035" />
+    <joint name="panda_finger_joint2" value="0.035" />
+  </group_state>
+  <group_state name="close" group="hand">
+    <joint name="panda_finger_joint1" value="0" />
+    <joint name="panda_finger_joint2" value="0" />
+  </group_state>
   <!--END EFFECTOR: Purpose: Represent information about an end effector.-->
   <end_effector name="hand" parent_link="panda_link8" group="hand" parent_group="panda_arm" />

Commit message: Add fully extended pose: 'home'

File: config/panda_arm_hand.srdf.xacro (robot description, xacro)
@@ -28,4 +28,13 @@
     <joint name="panda_joint7" value="0.785" />
   </group_state>
+  <group_state name="home" group="panda_arm_hand">
+    <joint name="panda_joint1" value="0" />
+    <joint name="panda_joint2" value="0" />
+    <joint name="panda_joint3" value="0" />
+    <joint name="panda_joint4" value="0" />
+    <joint name="panda_joint5" value="0" />
+    <joint name="panda_joint6" value="0" />
+    <joint name="panda_joint7" value="0.785" />
+  </group_state>
   <group_state name="open" group="hand">
     <joint name="panda_finger_joint1" value="0.035" />

Commit message: Add fully extended pose: 'extended' (#39)

File: config/panda_arm_hand.srdf.xacro (robot description, xacro)
@@ -28,4 +28,13 @@
     <joint name="panda_joint7" value="0.785" />
   </group_state>
+  <group_state name="extended" group="panda_arm_hand">
+    <joint name="panda_joint1" value="0" />
+    <joint name="panda_joint2" value="0" />
+    <joint name="panda_joint3" value="0" />
+    <joint name="panda_joint4" value="0" />
+    <joint name="panda_joint5" value="0" />
+    <joint name="panda_joint6" value="0" />
+    <joint name="panda_joint7" value="0.785" />
+  </group_state>
   <group_state name="open" group="hand">
     <joint name="panda_finger_joint1" value="0.035" />

Commit message: Update panda_arm_hand.srdf.xacro

File: config/panda_arm_hand.srdf.xacro (robot description, xacro)
@@ -27,4 +27,6 @@
     <joint name="panda_joint6" value="1.571" />
     <joint name="panda_joint7" value="0.785" />
+    <joint name="panda_finger_joint1" value="0" />
+    <joint name="panda_finger_joint2" value="0" />
   </group_state>
   <group_state name="extended" group="panda_arm_hand">
@@ -36,4 +38,6 @@
     <joint name="panda_joint6" value="0" />
     <joint name="panda_joint7" value="0.785" />
+    <joint name="panda_finger_joint1" value="0" />
+    <joint name="panda_finger_joint2" value="0" />
   </group_state>
   <group_state name="open" group="hand">

Commit message: add arm_group group_state names for kinetic

File: config/panda_arm_hand.srdf.xacro (robot description, xacro)
@@ -28,4 +28,21 @@
     <joint name="panda_joint7" value="0.785" />
   </group_state>
+  <group_state name="extended" group="panda_arm_hand">
+    <joint name="panda_joint1" value="0" />
+    <joint name="panda_joint2" value="0" />
+    <joint name="panda_joint3" value="0" />
+    <joint name="panda_joint4" value="0" />
+    <joint name="panda_joint5" value="0" />
+    <joint name="panda_joint6" value="0" />
+    <joint name="panda_joint7" value="0.785" />
+  </group_state>
+  <group_state name="open" group="hand">
+    <joint name="panda_finger_joint1" value="0.035" />
+    <joint name="panda_finger_joint2" value="0.035" />
+  </group_state>
+  <group_state name="close" group="hand">
+    <joint name="panda_finger_joint1" value="0" />
+    <joint name="panda_finger_joint2" value="0" />
+  </group_state>
   <!--END EFFECTOR: Purpose: Represent information about an end effector.-->
   <end_effector name="hand" parent_link="panda_link8" group="hand" parent_group="panda_arm" />

Commit message: Use predefined robot states from melodic-devel
Define poses ready, extended, open, close as in melodic-devel branch.

File: config/panda_arm_hand.srdf.xacro (robot description, xacro)
@@ -18,13 +18,11 @@
     <group name="hand" />
   </group>
-  <!--GROUP STATES: Purpose: Define a named state for a particular group, in terms of joint values. This is useful to define states like 'folded arms'-->
-  <group_state name="ready" group="panda_arm_hand">
-    <joint name="panda_joint1" value="0" />
-    <joint name="panda_joint2" value="-0.785" />
-    <joint name="panda_joint3" value="0" />
-    <joint name="panda_joint4" value="-2.356" />
-    <joint name="panda_joint5" value="0" />
-    <joint name="panda_joint6" value="1.571" />
-    <joint name="panda_joint7" value="0.785" />
+  <group_state name="open" group="hand">
+    <joint name="panda_finger_joint1" value="0.035" />
+    <joint name="panda_finger_joint2" value="0.035" />
+  </group_state>
+  <group_state name="close" group="hand">
+    <joint name="panda_finger_joint1" value="0" />
+    <joint name="panda_finger_joint2" value="0" />
   </group_state>
   <!--END EFFECTOR: Purpose: Represent information about an end effector.-->
