Commit message: Merge with panda_moveit_config from franka_ros

File: config/panda_arm.xacro (robot description, xacro)
@@ -1,8 +1,5 @@
 <?xml version="1.0" ?>
-<!--This does not replace URDF, and is not an extension of URDF.
-    This is a format for representing semantic information about the robot structure.
-    A URDF file must exist for this robot as well, where the joints and the links that are referenced are defined
--->
-<robot name="panda">
+<robot xmlns:xacro="http://www.ros.org/wiki/xacro" name="panda">
+  <xacro:macro name="panda_arm">
     <!--GROUPS: Representation of a set of joints and links. This can be useful for specifying DOF to plan for, defining arms, end effectors, etc-->
     <!--LINKS: When a link is specified, the parent joint of that link (if it exists) is automatically included-->
@@ -11,46 +8,38 @@
     <!--SUBGROUPS: Groups can also be formed by referencing to already defined group names-->
     <group name="panda_arm">
-        <joint name="virtual_joint" />
-        <joint name="panda_joint1" />
-        <joint name="panda_joint2" />
-        <joint name="panda_joint3" />
-        <joint name="panda_joint4" />
-        <joint name="panda_joint5" />
-        <joint name="panda_joint6" />
-        <joint name="panda_joint7" />
-        <joint name="panda_joint8" />
-    </group>
-    <group name="hand">
-        <link name="panda_hand" />
-        <link name="panda_leftfinger" />
-        <link name="panda_rightfinger" />
+      <link name="panda_link0" />
+      <link name="panda_link1" />
+      <link name="panda_link2" />
+      <link name="panda_link3" />
+      <link name="panda_link4" />
+      <link name="panda_link5" />
+      <link name="panda_link6" />
+      <link name="panda_link7" />
+      <link name="panda_link8" />
+      <joint name="virtual_joint" />
+      <joint name="panda_joint1" />
+      <joint name="panda_joint2" />
+      <joint name="panda_joint3" />
+      <joint name="panda_joint4" />
+      <joint name="panda_joint5" />
+      <joint name="panda_joint6" />
+      <joint name="panda_joint7" />
+      <joint name="panda_joint8" />
+      <chain base_link="panda_link0" tip_link="panda_link8" />
     </group>
     <!--GROUP STATES: Purpose: Define a named state for a particular group, in terms of joint values. This is useful to define states like 'folded arms'-->
-    <group_state name="home" group="panda_arm">
-        <joint name="panda_joint1" value="0" />
-        <joint name="panda_joint2" value="0" />
-        <joint name="panda_joint3" value="0" />
-        <joint name="panda_joint4" value="0" />
-        <joint name="panda_joint5" value="0" />
-        <joint name="panda_joint6" value="3.1416" />
-        <joint name="panda_joint7" value="1.5708" />
+    <group_state name="ready" group="panda_arm">
+      <joint name="panda_joint1" value="0" />
+      <joint name="panda_joint2" value="-0.785" />
+      <joint name="panda_joint3" value="0" />
+      <joint name="panda_joint4" value="-2.356" />
+      <joint name="panda_joint5" value="0" />
+      <joint name="panda_joint6" value="1.571" />
+      <joint name="panda_joint7" value="0.785" />
     </group_state>
     <!--END EFFECTOR: Purpose: Represent information about an end effector.-->
-    <end_effector name="eef" parent_link="panda_link8" group="hand" />
     <!--VIRTUAL JOINT: Purpose: this element defines a virtual joint between a robot link and an external frame of reference (considered fixed with respect to the robot)-->
     <virtual_joint name="virtual_joint" type="fixed" parent_frame="world" child_link="panda_link0" />
     <!--DISABLE COLLISIONS: By default it is assumed that any link of the robot could potentially come into collision with any other link in the robot. This tag disables collision checking between a specified pair of links. -->
-    <disable_collisions link1="panda_hand" link2="panda_leftfinger" reason="Adjacent" />
-    <disable_collisions link1="panda_hand" link2="panda_link3" reason="Never" />
-    <disable_collisions link1="panda_hand" link2="panda_link4" reason="Never" />
-    <disable_collisions link1="panda_hand" link2="panda_link5" reason="Default" />
-    <disable_collisions link1="panda_hand" link2="panda_link6" reason="Never" />
-    <disable_collisions link1="panda_hand" link2="panda_link7" reason="Adjacent" />
-    <disable_collisions link1="panda_hand" link2="panda_rightfinger" reason="Adjacent" />
-    <disable_collisions link1="panda_leftfinger" link2="panda_link3" reason="Never" />
-    <disable_collisions link1="panda_leftfinger" link2="panda_link4" reason="Never" />
-    <disable_collisions link1="panda_leftfinger" link2="panda_link6" reason="Never" />
-    <disable_collisions link1="panda_leftfinger" link2="panda_link7" reason="Never" />
-    <disable_collisions link1="panda_leftfinger" link2="panda_rightfinger" reason="Default" />
     <disable_collisions link1="panda_link0" link2="panda_link1" reason="Adjacent" />
     <disable_collisions link1="panda_link0" link2="panda_link2" reason="Never" />
@@ -67,13 +56,10 @@
     <disable_collisions link1="panda_link3" link2="panda_link6" reason="Never" />
     <disable_collisions link1="panda_link3" link2="panda_link7" reason="Never" />
-    <disable_collisions link1="panda_link3" link2="panda_rightfinger" reason="Never" />
     <disable_collisions link1="panda_link4" link2="panda_link5" reason="Adjacent" />
     <disable_collisions link1="panda_link4" link2="panda_link6" reason="Never" />
     <disable_collisions link1="panda_link4" link2="panda_link7" reason="Never" />
-    <disable_collisions link1="panda_link4" link2="panda_rightfinger" reason="Never" />
     <disable_collisions link1="panda_link5" link2="panda_link6" reason="Adjacent" />
     <disable_collisions link1="panda_link5" link2="panda_link7" reason="Default" />
     <disable_collisions link1="panda_link6" link2="panda_link7" reason="Adjacent" />
-    <disable_collisions link1="panda_link6" link2="panda_rightfinger" reason="Never" />
-    <disable_collisions link1="panda_link7" link2="panda_rightfinger" reason="Never" />
+  </xacro:macro>
 </robot>

Commit message: Simplify 'panda_arm' group

File: config/panda_arm.xacro (robot description, xacro)
@@ -8,22 +8,4 @@
     <!--SUBGROUPS: Groups can also be formed by referencing to already defined group names-->
     <group name="panda_arm">
-      <link name="panda_link0" />
-      <link name="panda_link1" />
-      <link name="panda_link2" />
-      <link name="panda_link3" />
-      <link name="panda_link4" />
-      <link name="panda_link5" />
-      <link name="panda_link6" />
-      <link name="panda_link7" />
-      <link name="panda_link8" />
-      <joint name="virtual_joint" />
-      <joint name="panda_joint1" />
-      <joint name="panda_joint2" />
-      <joint name="panda_joint3" />
-      <joint name="panda_joint4" />
-      <joint name="panda_joint5" />
-      <joint name="panda_joint6" />
-      <joint name="panda_joint7" />
-      <joint name="panda_joint8" />
       <chain base_link="panda_link0" tip_link="panda_link8" />
     </group>

Commit message: fix initial state of robot

File: config/panda_arm.xacro (robot description, xacro)
@@ -18,4 +18,13 @@
       <joint name="panda_joint5" value="0" />
       <joint name="panda_joint6" value="1.571" />
+      <joint name="panda_joint7" value="0.785" />
+    </group_state>
+    <group_state name="extended" group="panda_arm_hand">
+      <joint name="panda_joint1" value="0" />
+      <joint name="panda_joint2" value="0" />
+      <joint name="panda_joint3" value="0" />
+      <joint name="panda_joint4" value="0" />
+      <joint name="panda_joint5" value="0" />
+      <joint name="panda_joint6" value="0" />
       <joint name="panda_joint7" value="0.785" />
     </group_state>

File: config/panda_arm_hand.srdf.xacro (robot description, xacro)
@@ -18,23 +18,4 @@
     <group name="hand" />
   </group>
-  <!--GROUP STATES: Purpose: Define a named state for a particular group, in terms of joint values. This is useful to define states like 'folded arms'-->
-  <group_state name="ready" group="panda_arm_hand">
-    <joint name="panda_joint1" value="0" />
-    <joint name="panda_joint2" value="-0.785" />
-    <joint name="panda_joint3" value="0" />
-    <joint name="panda_joint4" value="-2.356" />
-    <joint name="panda_joint5" value="0" />
-    <joint name="panda_joint6" value="1.571" />
-    <joint name="panda_joint7" value="0.785" />
-  </group_state>
-  <group_state name="extended" group="panda_arm_hand">
-    <joint name="panda_joint1" value="0" />
-    <joint name="panda_joint2" value="0" />
-    <joint name="panda_joint3" value="0" />
-    <joint name="panda_joint4" value="0" />
-    <joint name="panda_joint5" value="0" />
-    <joint name="panda_joint6" value="0" />
-    <joint name="panda_joint7" value="0.785" />
-  </group_state>
   <group_state name="open" group="hand">
     <joint name="panda_finger_joint1" value="0.035" />

Commit message: moved named states to more meaningful groups

File: config/panda_arm.xacro (robot description, xacro)
@@ -18,4 +18,13 @@
       <joint name="panda_joint5" value="0" />
       <joint name="panda_joint6" value="1.571" />
+      <joint name="panda_joint7" value="0.785" />
+    </group_state>
+    <group_state name="extended" group="panda_arm">
+      <joint name="panda_joint1" value="0" />
+      <joint name="panda_joint2" value="0" />
+      <joint name="panda_joint3" value="0" />
+      <joint name="panda_joint4" value="0" />
+      <joint name="panda_joint5" value="0" />
+      <joint name="panda_joint6" value="0" />
       <joint name="panda_joint7" value="0.785" />
     </group_state>

File: config/panda_arm_hand.srdf.xacro (robot description, xacro)
@@ -27,13 +27,6 @@
     <joint name="panda_joint6" value="1.571" />
     <joint name="panda_joint7" value="0.785" />
-  </group_state>
-  <group_state name="extended" group="panda_arm_hand">
-    <joint name="panda_joint1" value="0" />
-    <joint name="panda_joint2" value="0" />
-    <joint name="panda_joint3" value="0" />
-    <joint name="panda_joint4" value="0" />
-    <joint name="panda_joint5" value="0" />
-    <joint name="panda_joint6" value="0" />
-    <joint name="panda_joint7" value="0.785" />
+    <joint name="panda_finger_joint1" value="0.035" />
+    <joint name="panda_finger_joint2" value="0.035" />
   </group_state>
   <group_state name="open" group="hand">

Commit message: update extended state with realistic values

File: config/panda_arm.xacro (robot description, xacro)
@@ -24,7 +24,7 @@
       <joint name="panda_joint2" value="0" />
       <joint name="panda_joint3" value="0" />
-      <joint name="panda_joint4" value="0" />
+      <joint name="panda_joint4" value="-0.0698" />
       <joint name="panda_joint5" value="0" />
-      <joint name="panda_joint6" value="0" />
+      <joint name="panda_joint6" value="3.14" />
       <joint name="panda_joint7" value="0.785" />
     </group_state>

Commit message: Add tranposrt joint state

File: config/panda_arm.xacro (robot description, xacro)
@@ -29,4 +29,13 @@
       <joint name="panda_joint7" value="0.785" />
     </group_state>
+    <group_state name="transport" group="panda_arm">
+      <joint name="panda_joint1" value="0" />
+      <joint name="panda_joint2" value="-0.5599" />
+      <joint name="panda_joint3" value="0" />
+      <joint name="panda_joint4" value="-2.97" />
+      <joint name="panda_joint5" value="0" />
+      <joint name="panda_joint6" value="0" />
+      <joint name="panda_joint7" value="0.785" />
+    </group_state>
     <!--END EFFECTOR: Purpose: Represent information about an end effector.-->
     <!--VIRTUAL JOINT: Purpose: this element defines a virtual joint between a robot link and an external frame of reference (considered fixed with respect to the robot)-->

Commit message: Generated using the latest features from MoveIt

File: config/panda_arm.xacro (robot description, xacro)
@@ -12,29 +12,20 @@
     <!--GROUP STATES: Purpose: Define a named state for a particular group, in terms of joint values. This is useful to define states like 'folded arms'-->
     <group_state name="ready" group="panda_arm">
-      <joint name="panda_joint1" value="0" />
-      <joint name="panda_joint2" value="-0.785" />
-      <joint name="panda_joint3" value="0" />
-      <joint name="panda_joint4" value="-2.356" />
-      <joint name="panda_joint5" value="0" />
-      <joint name="panda_joint6" value="1.571" />
-      <joint name="panda_joint7" value="0.785" />
+        <joint name="panda_joint1" value="0"/>
+        <joint name="panda_joint2" value="-0.785"/>
+        <joint name="panda_joint3" value="0"/>
+        <joint name="panda_joint4" value="-2.356"/>
+        <joint name="panda_joint5" value="0"/>
+        <joint name="panda_joint6" value="1.571"/>
+        <joint name="panda_joint7" value="-0.7855"/>
     </group_state>
     <group_state name="extended" group="panda_arm">
-      <joint name="panda_joint1" value="0" />
-      <joint name="panda_joint2" value="0" />
-      <joint name="panda_joint3" value="0" />
-      <joint name="panda_joint4" value="0" />
-      <joint name="panda_joint5" value="0" />
-      <joint name="panda_joint6" value="0" />
-      <joint name="panda_joint7" value="0.785" />
-    </group_state>
-    <group_state name="transport" group="panda_arm">
-      <joint name="panda_joint1" value="0" />
-      <joint name="panda_joint2" value="-0.5599" />
-      <joint name="panda_joint3" value="0" />
-      <joint name="panda_joint4" value="-2.97" />
-      <joint name="panda_joint5" value="0" />
-      <joint name="panda_joint6" value="0" />
-      <joint name="panda_joint7" value="0.785" />
+        <joint name="panda_joint1" value="0"/>
+        <joint name="panda_joint2" value="-0.3927"/>
+        <joint name="panda_joint3" value="0"/>
+        <joint name="panda_joint4" value="-0.7855"/>
+        <joint name="panda_joint5" value="0"/>
+        <joint name="panda_joint6" value="3.142"/>
+        <joint name="panda_joint7" value="-0.785"/>
     </group_state>
     <!--END EFFECTOR: Purpose: Represent information about an end effector.-->

Commit message: Disable collision between panda_link8 & panda_link6 + panda_link7

File: config/panda_arm.xacro (robot description, xacro)
@@ -18,5 +18,5 @@
         <joint name="panda_joint5" value="0"/>
         <joint name="panda_joint6" value="1.571"/>
-        <joint name="panda_joint7" value="-0.7855"/>
+        <joint name="panda_joint7" value="0.785"/>
     </group_state>
     <group_state name="extended" group="panda_arm">
@@ -50,5 +50,7 @@
     <disable_collisions link1="panda_link5" link2="panda_link6" reason="Adjacent" />
     <disable_collisions link1="panda_link5" link2="panda_link7" reason="Default" />
+    <disable_collisions link1="panda_link5" link2="panda_link8" reason="Default" />
     <disable_collisions link1="panda_link6" link2="panda_link7" reason="Adjacent" />
+    <disable_collisions link1="panda_link6" link2="panda_link8" reason="Default" />
     <disable_collisions link1="panda_link7" link2="panda_link8" reason="Adjacent" />
   </xacro:macro>
