Commit message: Add demo_gazebo.launch using franka_gazebo
This commit adds demo_gazebo.launch using the gazebo simulation of the franka_gazebo package
Additionally, the virtual_joint is removed from the move group definition.

File: config/panda_arm.xacro (robot description, xacro)
@@ -1,64 +1,67 @@
 <?xml version="1.0" ?>
 <robot xmlns:xacro="http://www.ros.org/wiki/xacro" name="panda">
-  <xacro:macro name="panda_arm">
-    <!--GROUPS: Representation of a set of joints and links. This can be useful for specifying DOF to plan for, defining arms, end effectors, etc-->
-    <!--LINKS: When a link is specified, the parent joint of that link (if it exists) is automatically included-->
-    <!--JOINTS: When a joint is specified, the child link of that joint (which will always exist) is automatically included-->
-    <!--CHAINS: When a chain is specified, all the links along the chain (including endpoints) are included in the group. Additionally, all the joints that are parents to included links are also included. This means that joints along the chain and the parent joint of the base link are included in the group-->
-    <!--SUBGROUPS: Groups can also be formed by referencing to already defined group names-->
-    <group name="panda_arm">
-      <chain base_link="panda_link0" tip_link="panda_link8" />
-    </group>
-    <!--GROUP STATES: Purpose: Define a named state for a particular group, in terms of joint values. This is useful to define states like 'folded arms'-->
-    <group_state name="ready" group="panda_arm">
-      <joint name="panda_joint1" value="0" />
-      <joint name="panda_joint2" value="-0.785" />
-      <joint name="panda_joint3" value="0" />
-      <joint name="panda_joint4" value="-2.356" />
-      <joint name="panda_joint5" value="0" />
-      <joint name="panda_joint6" value="1.571" />
-      <joint name="panda_joint7" value="0.785" />
-    </group_state>
-    <group_state name="extended" group="panda_arm">
-      <joint name="panda_joint1" value="0" />
-      <joint name="panda_joint2" value="0" />
-      <joint name="panda_joint3" value="0" />
-      <joint name="panda_joint4" value="0" />
-      <joint name="panda_joint5" value="0" />
-      <joint name="panda_joint6" value="0" />
-      <joint name="panda_joint7" value="0.785" />
-    </group_state>
-    <group_state name="transport" group="panda_arm">
-      <joint name="panda_joint1" value="0" />
-      <joint name="panda_joint2" value="-0.5599" />
-      <joint name="panda_joint3" value="0" />
-      <joint name="panda_joint4" value="-2.97" />
-      <joint name="panda_joint5" value="0" />
-      <joint name="panda_joint6" value="0" />
-      <joint name="panda_joint7" value="0.785" />
-    </group_state>
-    <!--END EFFECTOR: Purpose: Represent information about an end effector.-->
-    <!--VIRTUAL JOINT: Purpose: this element defines a virtual joint between a robot link and an external frame of reference (considered fixed with respect to the robot)-->
-    <virtual_joint name="virtual_joint" type="floating" parent_frame="world" child_link="panda_link0" />
-    <!--DISABLE COLLISIONS: By default it is assumed that any link of the robot could potentially come into collision with any other link in the robot. This tag disables collision checking between a specified pair of links. -->
-    <disable_collisions link1="panda_link0" link2="panda_link1" reason="Adjacent" />
-    <disable_collisions link1="panda_link0" link2="panda_link2" reason="Never" />
-    <disable_collisions link1="panda_link0" link2="panda_link3" reason="Never" />
-    <disable_collisions link1="panda_link0" link2="panda_link4" reason="Never" />
-    <disable_collisions link1="panda_link1" link2="panda_link2" reason="Adjacent" />
-    <disable_collisions link1="panda_link1" link2="panda_link3" reason="Default" />
-    <disable_collisions link1="panda_link1" link2="panda_link4" reason="Never" />
-    <disable_collisions link1="panda_link2" link2="panda_link3" reason="Adjacent" />
-    <disable_collisions link1="panda_link2" link2="panda_link4" reason="Never" />
-    <disable_collisions link1="panda_link3" link2="panda_link4" reason="Adjacent" />
-    <disable_collisions link1="panda_link3" link2="panda_link6" reason="Never" />
-    <disable_collisions link1="panda_link4" link2="panda_link5" reason="Adjacent" />
-    <disable_collisions link1="panda_link4" link2="panda_link6" reason="Never" />
-    <disable_collisions link1="panda_link4" link2="panda_link7" reason="Never" />
-    <disable_collisions link1="panda_link4" link2="panda_link8" reason="Never" />
-    <disable_collisions link1="panda_link5" link2="panda_link6" reason="Adjacent" />
-    <disable_collisions link1="panda_link6" link2="panda_link7" reason="Adjacent" />
-    <disable_collisions link1="panda_link6" link2="panda_link8" reason="Default" />
-    <disable_collisions link1="panda_link7" link2="panda_link8" reason="Adjacent" />
-  </xacro:macro>
+    <xacro:macro name="panda_arm">
+        <!--GROUPS: Representation of a set of joints and links. This can be useful for specifying DOF to plan for, defining arms, end effectors, etc-->
+        <!--LINKS: When a link is specified, the parent joint of that link (if it exists) is automatically included-->
+        <!--JOINTS: When a joint is specified, the child link of that joint (which will always exist) is automatically included-->
+        <!--CHAINS: When a chain is specified, all the links along the chain (including endpoints) are included in the group. Additionally, all the joints that are parents to included links are also included. This means that joints along the chain and the parent joint of the base link are included in the group-->
+        <!--SUBGROUPS: Groups can also be formed by referencing to already defined group names-->
+        <group name="panda_arm">
+            <joint name="panda_joint1"/>
+            <joint name="panda_joint2"/>
+            <joint name="panda_joint3"/>
+            <joint name="panda_joint4"/>
+            <joint name="panda_joint5"/>
+            <joint name="panda_joint6"/>
+            <joint name="panda_joint7"/>
+            <joint name="panda_joint8"/>
+        </group>
+        <!--GROUP STATES: Purpose: Define a named state for a particular group, in terms of joint values. This is useful to define states like 'folded arms'-->
+        <group_state name="ready" group="panda_arm">
+            <joint name="panda_joint1" value="0"/>
+            <joint name="panda_joint2" value="-0.785"/>
+            <joint name="panda_joint3" value="0"/>
+            <joint name="panda_joint4" value="-2.356"/>
+            <joint name="panda_joint5" value="0"/>
+            <joint name="panda_joint6" value="1.571"/>
+            <joint name="panda_joint7" value="-0.7855"/>
+        </group_state>
+        <group_state name="extended" group="panda_arm">
+            <joint name="panda_joint1" value="0"/>
+            <joint name="panda_joint2" value="-0.3927"/>
+            <joint name="panda_joint3" value="0"/>
+            <joint name="panda_joint4" value="-0.7855"/>
+            <joint name="panda_joint5" value="0"/>
+            <joint name="panda_joint6" value="3.142"/>
+            <joint name="panda_joint7" value="-0.785"/>
+        </group_state>
+        <!--VIRTUAL JOINT: Purpose: this element defines a virtual joint between a robot link and an external frame of reference (considered fixed with respect to the robot)-->
+        <virtual_joint name="virtual_joint" type="fixed" parent_frame="world" child_link="panda_link0"/>
+        <!--DISABLE COLLISIONS: By default it is assumed that any link of the robot could potentially come into collision with any other link in the robot. This tag disables collision checking between a specified pair of links. -->
+        <disable_collisions link1="panda_link0" link2="panda_link1" reason="Adjacent"/>
+        <disable_collisions link1="panda_link0" link2="panda_link2" reason="Never"/>
+        <disable_collisions link1="panda_link0" link2="panda_link3" reason="Never"/>
+        <disable_collisions link1="panda_link0" link2="panda_link4" reason="Never"/>
+        <disable_collisions link1="panda_link1" link2="panda_link2" reason="Adjacent"/>
+        <disable_collisions link1="panda_link1" link2="panda_link3" reason="Default"/>
+        <disable_collisions link1="panda_link1" link2="panda_link4" reason="Never"/>
+        <disable_collisions link1="panda_link2" link2="panda_link3" reason="Adjacent"/>
+        <disable_collisions link1="panda_link2" link2="panda_link4" reason="Never"/>
+        <disable_collisions link1="panda_link3" link2="panda_link4" reason="Adjacent"/>
+        <disable_collisions link1="panda_link3" link2="panda_link6" reason="Never"/>
+        <disable_collisions link1="panda_link4" link2="panda_link5" reason="Adjacent"/>
+        <disable_collisions link1="panda_link4" link2="panda_link6" reason="Never"/>
+        <disable_collisions link1="panda_link4" link2="panda_link7" reason="Never"/>
+        <disable_collisions link1="panda_link4" link2="panda_link8" reason="Never"/>
+        <disable_collisions link1="panda_link5" link2="panda_link6" reason="Adjacent"/>
+        <disable_collisions link1="panda_link5" link2="panda_link7" reason="Default"/>
+        <disable_collisions link1="panda_link6" link2="panda_link7" reason="Adjacent"/>
+        <disable_collisions link1="panda_link7" link2="panda_link8" reason="Adjacent"/>
+        <!-- Fix self-collisions between too coarse collision geometries provided by franka_description
+             See https://github.com/ros-planning/panda_moveit_config/issues/72#issuecomment-768472329
+                 https://github.com/ros-planning/panda_moveit_config/pull/35#pullrequestreview-390715967
+        -->
+        <disable_collisions link1="panda_link5" link2="panda_link8" reason="Default" />
+        <disable_collisions link1="panda_link6" link2="panda_link8" reason="Default"/>
+    </xacro:macro>
 </robot>

Commit message: Add demo_gazebo.launch using franka_gazebo
This commit adds demo_gazebo.launch using the gazebo simulation of the franka_gazebo package
Additionally, the virtual_joint is removed from the move group definition.

File: config/panda_arm.xacro (robot description, xacro)
@@ -8,5 +8,4 @@
         <!--SUBGROUPS: Groups can also be formed by referencing to already defined group names-->
         <group name="panda_arm">
-            <joint name="virtual_joint"/>
             <joint name="panda_joint1"/>
             <joint name="panda_joint2"/>

Commit message: SRDF: Use chain specification

File: config/panda_arm.xacro (robot description, xacro)
@@ -8,12 +8,5 @@
         <!--SUBGROUPS: Groups can also be formed by referencing to already defined group names-->
         <group name="panda_arm">
-            <joint name="panda_joint1"/>
-            <joint name="panda_joint2"/>
-            <joint name="panda_joint3"/>
-            <joint name="panda_joint4"/>
-            <joint name="panda_joint5"/>
-            <joint name="panda_joint6"/>
-            <joint name="panda_joint7"/>
-            <joint name="panda_joint8"/>
+            <chain base_link="panda_link0" tip_link="panda_link8"/>
         </group>
         <!--GROUP STATES: Purpose: Define a named state for a particular group, in terms of joint values. This is useful to define states like 'folded arms'-->

Commit message: Fix group states
- Use factors of pi
- Fix joint limit violation for "extended" pose

File: config/panda_arm.xacro (robot description, xacro)
@@ -12,20 +12,20 @@
         <!--GROUP STATES: Purpose: Define a named state for a particular group, in terms of joint values. This is useful to define states like 'folded arms'-->
         <group_state name="ready" group="panda_arm">
-            <joint name="panda_joint1" value="0"/>
-            <joint name="panda_joint2" value="-0.785"/>
-            <joint name="panda_joint3" value="0"/>
-            <joint name="panda_joint4" value="-2.356"/>
-            <joint name="panda_joint5" value="0"/>
-            <joint name="panda_joint6" value="1.571"/>
-            <joint name="panda_joint7" value="0.785"/>
+            <joint name="panda_joint1" value="0" />
+            <joint name="panda_joint2" value="${-pi/4}" />
+            <joint name="panda_joint3" value="0" />
+            <joint name="panda_joint4" value="${-3*pi/4}" />
+            <joint name="panda_joint5" value="0" />
+            <joint name="panda_joint6" value="${pi/2}" />
+            <joint name="panda_joint7" value="${pi/4}" />
         </group_state>
         <group_state name="extended" group="panda_arm">
-            <joint name="panda_joint1" value="0"/>
-            <joint name="panda_joint2" value="0"/>
-            <joint name="panda_joint3" value="0"/>
-            <joint name="panda_joint4" value="0"/>
-            <joint name="panda_joint5" value="0"/>
-            <joint name="panda_joint6" value="0"/>
-            <joint name="panda_joint7" value="0.785"/>
+            <joint name="panda_joint1" value="0" />
+            <joint name="panda_joint2" value="0" />
+            <joint name="panda_joint3" value="0" />
+            <joint name="panda_joint4" value="-0.1" />
+            <joint name="panda_joint5" value="0" />
+            <joint name="panda_joint6" value="${pi}" />
+            <joint name="panda_joint7" value="${pi/4}" />
         </group_state>
         <!--VIRTUAL JOINT: Purpose: this element defines a virtual joint between a robot link and an external frame of reference (considered fixed with respect to the robot)-->

Commit message: Fix group states
- Use factors of pi
- Fix joint limit violation for "extended" pose

File: config/panda_arm.xacro (robot description, xacro)
@@ -12,20 +12,20 @@
         <!--GROUP STATES: Purpose: Define a named state for a particular group, in terms of joint values. This is useful to define states like 'folded arms'-->
         <group_state name="ready" group="panda_arm">
-            <joint name="panda_joint1" value="0"/>
-            <joint name="panda_joint2" value="-0.785"/>
-            <joint name="panda_joint3" value="0"/>
-            <joint name="panda_joint4" value="-2.356"/>
-            <joint name="panda_joint5" value="0"/>
-            <joint name="panda_joint6" value="1.571"/>
-            <joint name="panda_joint7" value="-0.7855"/>
+            <joint name="panda_joint1" value="0" />
+            <joint name="panda_joint2" value="${-pi/4}" />
+            <joint name="panda_joint3" value="0" />
+            <joint name="panda_joint4" value="${-3*pi/4}" />
+            <joint name="panda_joint5" value="0" />
+            <joint name="panda_joint6" value="${pi/2}" />
+            <joint name="panda_joint7" value="${pi/4}" />
         </group_state>
         <group_state name="extended" group="panda_arm">
-            <joint name="panda_joint1" value="0"/>
-            <joint name="panda_joint2" value="-0.3927"/>
-            <joint name="panda_joint3" value="0"/>
-            <joint name="panda_joint4" value="-0.7855"/>
-            <joint name="panda_joint5" value="0"/>
-            <joint name="panda_joint6" value="3.142"/>
-            <joint name="panda_joint7" value="-0.785"/>
+            <joint name="panda_joint1" value="0" />
+            <joint name="panda_joint2" value="0" />
+            <joint name="panda_joint3" value="0" />
+            <joint name="panda_joint4" value="-0.1" />
+            <joint name="panda_joint5" value="0" />
+            <joint name="panda_joint6" value="${pi/2}" />
+            <joint name="panda_joint7" value="${pi/4}" />
         </group_state>
         <!--VIRTUAL JOINT: Purpose: this element defines a virtual joint between a robot link and an external frame of reference (considered fixed with respect to the robot)-->
@@ -55,5 +55,5 @@
                  https://github.com/ros-planning/panda_moveit_config/pull/35#pullrequestreview-390715967
         -->
-        <disable_collisions link1="panda_link5" link2="panda_link8" reason="Default" />
+        <disable_collisions link1="panda_link5" link2="panda_link8" reason="Default"/>
         <disable_collisions link1="panda_link6" link2="panda_link8" reason="Default"/>
     </xacro:macro>

Commit message: fix collison links and group states

File: config/panda_arm.xacro (robot description, xacro)
@@ -1,3 +1,3 @@
-<?xml version="1.0" ?>
+<?xml version="1.0"?>
 <robot xmlns:xacro="http://www.ros.org/wiki/xacro" name="panda">
   <xacro:macro name="panda_arm">
@@ -13,10 +13,10 @@
     <group_state name="ready" group="panda_arm">
       <joint name="panda_joint1" value="0" />
-      <joint name="panda_joint2" value="-0.785" />
+      <joint name="panda_joint2" value="${-pi/4}" />
       <joint name="panda_joint3" value="0" />
-      <joint name="panda_joint4" value="-2.356" />
+      <joint name="panda_joint4" value="${-3*pi/4}" />
       <joint name="panda_joint5" value="0" />
-      <joint name="panda_joint6" value="1.571" />
-      <joint name="panda_joint7" value="0.785" />
+      <joint name="panda_joint6" value="${pi/2}" />
+      <joint name="panda_joint7" value="${pi/4}" />
     </group_state>
     <group_state name="extended" group="panda_arm">
@@ -24,21 +24,12 @@
       <joint name="panda_joint2" value="0" />
       <joint name="panda_joint3" value="0" />
-      <joint name="panda_joint4" value="0" />
+      <joint name="panda_joint4" value="-0.1" />
       <joint name="panda_joint5" value="0" />
-      <joint name="panda_joint6" value="0" />
-      <joint name="panda_joint7" value="0.785" />
-    </group_state>
-    <group_state name="transport" group="panda_arm">
-      <joint name="panda_joint1" value="0" />
-      <joint name="panda_joint2" value="-0.5599" />
-      <joint name="panda_joint3" value="0" />
-      <joint name="panda_joint4" value="-2.97" />
-      <joint name="panda_joint5" value="0" />
-      <joint name="panda_joint6" value="0" />
-      <joint name="panda_joint7" value="0.785" />
+      <joint name="panda_joint6" value="${pi/2}" />
+      <joint name="panda_joint7" value="${pi/4}" />
     </group_state>
     <!--END EFFECTOR: Purpose: Represent information about an end effector.-->
     <!--VIRTUAL JOINT: Purpose: this element defines a virtual joint between a robot link and an external frame of reference (considered fixed with respect to the robot)-->
-    <virtual_joint name="virtual_joint" type="floating" parent_frame="world" child_link="panda_link0" />
+    <virtual_joint name="virtual_joint" type="fixed" parent_frame="world" child_link="panda_link0" />
     <!--DISABLE COLLISIONS: By default it is assumed that any link of the robot could potentially come into collision with any other link in the robot. This tag disables collision checking between a specified pair of links. -->
     <disable_collisions link1="panda_link0" link2="panda_link1" reason="Adjacent" />
@@ -52,4 +43,5 @@
     <disable_collisions link1="panda_link2" link2="panda_link4" reason="Never" />
     <disable_collisions link1="panda_link3" link2="panda_link4" reason="Adjacent" />
+    <disable_collisions link1="panda_link3" link2="panda_link5" reason="Default" />
     <disable_collisions link1="panda_link3" link2="panda_link6" reason="Never" />
     <disable_collisions link1="panda_link4" link2="panda_link5" reason="Adjacent" />
@@ -58,7 +50,13 @@
     <disable_collisions link1="panda_link4" link2="panda_link8" reason="Never" />
     <disable_collisions link1="panda_link5" link2="panda_link6" reason="Adjacent" />
+    <disable_collisions link1="panda_link5" link2="panda_link7" reason="Default" />
     <disable_collisions link1="panda_link6" link2="panda_link7" reason="Adjacent" />
+    <disable_collisions link1="panda_link7" link2="panda_link8" reason="Adjacent" />
+    <!-- Fix self-collisions between too coarse collision geometries provided by franka_description
+             See https://github.com/ros-planning/panda_moveit_config/issues/72#issuecomment-768472329
+                 https://github.com/ros-planning/panda_moveit_config/pull/35#pullrequestreview-390715967
+        -->
+    <disable_collisions link1="panda_link5" link2="panda_link8" reason="Default" />
     <disable_collisions link1="panda_link6" link2="panda_link8" reason="Default" />
-    <disable_collisions link1="panda_link7" link2="panda_link8" reason="Adjacent" />
   </xacro:macro>
 </robot>
