Commit message: Added tcp_joint to config files

File: config/hand.xacro (robot description, xacro)
@@ -13,4 +13,5 @@
       <joint name="panda_finger_joint1" />
       <passive_joint name="panda_finger_joint2" />
+      <link name="panda_tcp" />
     </group>
     <!--GROUP STATES: Purpose: Define a named state for a particular group, in terms of joint values. This is useful to define states like 'folded arms'-->

File: config/panda_arm_hand.srdf.xacro (robot description, xacro)
@@ -28,4 +28,5 @@
   <!--END EFFECTOR: Purpose: Represent information about an end effector.-->
   <end_effector name="hand" parent_link="panda_link8" group="hand" parent_group="panda_arm" />
+  <end_effector name="tcp" parent_link="panda_tcp" group="panda_arm" parent_group="hand" />
   <!--DISABLE COLLISIONS: By default it is assumed that any link of the robot could potentially come into collision with any other link in the robot. This tag disables collision checking between a specified pair of links. -->
   <disable_collisions link1="panda_hand" link2="panda_link4" reason="Never" />

Commit message: Rework collision models for hand
... utilizing a new feature of MoveIt / SRDF
Now, it's possible to disable collision for a specific collision name by default.
The definition of specific collision pairs will override this default.

This allows disabling collision for the coarse hand geometries
and enabling it for selected pairs of links only (for self-collision checking).

On the other hand, the detailed hand collision geometries are enabled by default,
but selectively disabled for self-collision checking for all arm links.

File: config/hand.xacro (robot description, xacro)
@@ -1,4 +1,19 @@
 <?xml version="1.0" encoding="UTF-8"?>
 <robot xmlns:xacro="http://www.ros.org/wiki/xacro" name="panda">
+    <xacro:macro name="finger_collisions" params="finger">
+        <!-- Disable all self-collisions between finger and arm links,
+             as these are already covered by the coarser hand collision model -->
+        <disable_collisions link1="${finger}" link2="panda_link0" reason="Default" />
+        <disable_collisions link1="${finger}" link2="panda_link1" reason="Default" />
+        <disable_collisions link1="${finger}" link2="panda_link2" reason="Default" />
+        <disable_collisions link1="${finger}" link2="panda_link3" reason="Default" />
+        <disable_collisions link1="${finger}" link2="panda_link4" reason="Default" />
+        <disable_collisions link1="${finger}" link2="panda_link5" reason="Default" />
+        <disable_collisions link1="${finger}" link2="panda_link6" reason="Default" />
+        <disable_collisions link1="${finger}" link2="panda_link7" reason="Default" />
+        <disable_collisions link1="${finger}" link2="panda_link8" reason="Default" />
+        <disable_collisions link1="${finger}" link2="panda_hand" reason="Default" />
+        <disable_collisions link1="${finger}" link2="panda_hand_coarse" reason="Default" />
+    </xacro:macro>
     <xacro:macro name="hand">
         <!--GROUPS: Representation of a set of joints and links. This can be useful for specifying DOF to plan for, defining arms, end effectors, etc-->
@@ -8,4 +23,5 @@
         <!--SUBGROUPS: Groups can also be formed by referencing to already defined group names-->
         <group name="hand">
+            <link name="panda_hand_coarse" />
             <link name="panda_hand"/>
             <link name="panda_leftfinger"/>
@@ -25,22 +41,14 @@
         <!--PASSIVE JOINT: Purpose: this element is used to mark joints that are not actuated-->
         <!--DISABLE COLLISIONS: By default it is assumed that any link of the robot could potentially come into collision with any other link in the robot. This tag disables collision checking between a specified pair of links. -->
-        <disable_collisions link1="panda_hand" link2="panda_leftfinger" reason="Adjacent"/>
-        <disable_collisions link1="panda_hand" link2="panda_link4" reason="Never"/>
-        <disable_collisions link1="panda_hand" link2="panda_link5" reason="Default"/>
-        <disable_collisions link1="panda_hand" link2="panda_link6" reason="Never"/>
-        <disable_collisions link1="panda_hand" link2="panda_link7" reason="Default"/>
-        <disable_collisions link1="panda_hand" link2="panda_link8" reason="Adjacent"/>
-        <disable_collisions link1="panda_hand" link2="panda_rightfinger" reason="Adjacent"/>
-        <disable_collisions link1="panda_leftfinger" link2="panda_link4" reason="Never"/>
-        <disable_collisions link1="panda_leftfinger" link2="panda_link5" reason="Default"/>
-        <disable_collisions link1="panda_leftfinger" link2="panda_link6" reason="Never"/>
-        <disable_collisions link1="panda_leftfinger" link2="panda_link7" reason="Never"/>
-        <disable_collisions link1="panda_leftfinger" link2="panda_link8" reason="Never"/>
-        <disable_collisions link1="panda_leftfinger" link2="panda_rightfinger" reason="Default"/>
-        <disable_collisions link1="panda_link4" link2="panda_rightfinger" reason="Never"/>
-        <disable_collisions link1="panda_link5" link2="panda_rightfinger" reason="Default"/>
-        <disable_collisions link1="panda_link6" link2="panda_rightfinger" reason="Never"/>
-        <disable_collisions link1="panda_link7" link2="panda_rightfinger" reason="Never"/>
-        <disable_collisions link1="panda_link8" link2="panda_rightfinger" reason="Never"/>
+        <collision_default link="panda_hand_coarse" allow="ALWAYS" />
+        <enable_collisions link1="panda_hand_coarse" link2="panda_link0" />
+        <enable_collisions link1="panda_hand_coarse" link2="panda_link1" />
+        <enable_collisions link1="panda_hand_coarse" link2="panda_link2" />
+        <enable_collisions link1="panda_hand_coarse" link2="panda_link3" />
+        <disable_collisions link1="panda_hand" link2="panda_link7" />
+        <disable_collisions link1="panda_hand" link2="panda_link8" />
+        <xacro:finger_collisions finger="panda_leftfinger" />
+        <xacro:finger_collisions finger="panda_rightfinger" />
+        <disable_collisions link1="panda_leftfinger" link2="panda_rightfinger" reason="Default" />
     </xacro:macro>
 </robot>

Commit message: Rework collision models for hand
... utilizing a new feature of MoveIt / SRDF
Now, it's possible to disable collision for a specific collision name by default.
The definition of specific collision pairs will override this default.

This allows disabling collision for the coarse hand geometries
and enabling it for selected pairs of links only (for self-collision checking).

On the other hand, the detailed hand collision geometries are enabled by default,
but selectively disabled for self-collision checking for all arm links.

File: config/hand.xacro (robot description, xacro)
@@ -1,4 +1,19 @@
 <?xml version="1.0" encoding="UTF-8"?>
 <robot xmlns:xacro="http://www.ros.org/wiki/xacro" name="panda">
+    <xacro:macro name="finger_collisions" params="finger">
+        <!-- Disable all self-collisions between finger and arm links,
+             as these are already covered by the coarser hand collision model -->
+        <disable_collisions link1="${finger}" link2="panda_link0" reason="Default" />
+        <disable_collisions link1="${finger}" link2="panda_link1" reason="Default" />
+        <disable_collisions link1="${finger}" link2="panda_link2" reason="Default" />
+        <disable_collisions link1="${finger}" link2="panda_link3" reason="Default" />
+        <disable_collisions link1="${finger}" link2="panda_link4" reason="Default" />
+        <disable_collisions link1="${finger}" link2="panda_link5" reason="Default" />
+        <disable_collisions link1="${finger}" link2="panda_link6" reason="Default" />
+        <disable_collisions link1="${finger}" link2="panda_link7" reason="Default" />
+        <disable_collisions link1="${finger}" link2="panda_link8" reason="Default" />
+        <disable_collisions link1="${finger}" link2="panda_hand" reason="Default" />
+        <disable_collisions link1="${finger}" link2="panda_hand_coarse" reason="Default" />
+    </xacro:macro>
     <xacro:macro name="hand">
         <!--GROUPS: Representation of a set of joints and links. This can be useful for specifying DOF to plan for, defining arms, end effectors, etc-->
@@ -8,4 +23,5 @@
         <!--SUBGROUPS: Groups can also be formed by referencing to already defined group names-->
         <group name="hand">
+            <link name="panda_hand_coarse" />
             <link name="panda_hand"/>
             <link name="panda_leftfinger"/>
@@ -26,22 +42,14 @@
         <passive_joint name="panda_finger_joint2"/>
         <!--DISABLE COLLISIONS: By default it is assumed that any link of the robot could potentially come into collision with any other link in the robot. This tag disables collision checking between a specified pair of links. -->
-        <disable_collisions link1="panda_hand" link2="panda_leftfinger" reason="Adjacent"/>
-        <disable_collisions link1="panda_hand" link2="panda_link4" reason="Never"/>
-        <disable_collisions link1="panda_hand" link2="panda_link5" reason="Default"/>
-        <disable_collisions link1="panda_hand" link2="panda_link6" reason="Never"/>
-        <disable_collisions link1="panda_hand" link2="panda_link7" reason="Default"/>
-        <disable_collisions link1="panda_hand" link2="panda_link8" reason="Adjacent"/>
-        <disable_collisions link1="panda_hand" link2="panda_rightfinger" reason="Adjacent"/>
-        <disable_collisions link1="panda_leftfinger" link2="panda_link4" reason="Never"/>
-        <disable_collisions link1="panda_leftfinger" link2="panda_link5" reason="Default"/>
-        <disable_collisions link1="panda_leftfinger" link2="panda_link6" reason="Never"/>
-        <disable_collisions link1="panda_leftfinger" link2="panda_link7" reason="Never"/>
-        <disable_collisions link1="panda_leftfinger" link2="panda_link8" reason="Never"/>
-        <disable_collisions link1="panda_leftfinger" link2="panda_rightfinger" reason="Default"/>
-        <disable_collisions link1="panda_link4" link2="panda_rightfinger" reason="Never"/>
-        <disable_collisions link1="panda_link5" link2="panda_rightfinger" reason="Default"/>
-        <disable_collisions link1="panda_link6" link2="panda_rightfinger" reason="Never"/>
-        <disable_collisions link1="panda_link7" link2="panda_rightfinger" reason="Never"/>
-        <disable_collisions link1="panda_link8" link2="panda_rightfinger" reason="Never"/>
+        <collision_default link="panda_hand_coarse" allow="ALWAYS" />
+        <enable_collisions link1="panda_hand_coarse" link2="panda_link0" />
+        <enable_collisions link1="panda_hand_coarse" link2="panda_link1" />
+        <enable_collisions link1="panda_hand_coarse" link2="panda_link2" />
+        <enable_collisions link1="panda_hand_coarse" link2="panda_link3" />
+        <disable_collisions link1="panda_hand" link2="panda_link7" />
+        <disable_collisions link1="panda_hand" link2="panda_link8" />
+        <xacro:finger_collisions finger="panda_leftfinger" />
+        <xacro:finger_collisions finger="panda_rightfinger" />
+        <disable_collisions link1="panda_leftfinger" link2="panda_rightfinger" reason="Default" />
     </xacro:macro>
 </robot>

Commit message: Remove panda_hand_coarse from hand group
We don't want to consider the coarse model for any environmental interaction.
MoveIt Task Constructor uses the group to disable and re-enable collisions
when grasping resp. releasing an object.

File: config/hand.xacro (robot description, xacro)
@@ -23,5 +23,4 @@
         <!--SUBGROUPS: Groups can also be formed by referencing to already defined group names-->
         <group name="hand">
-            <link name="panda_hand_coarse" />
             <link name="panda_hand"/>
             <link name="panda_leftfinger"/>
