Commit message: Maintain compatibility with old panda_arm group and its panda_link8 tip
Introduce a new, second arm group, "arm", which defines the new tool tip.
A corresponding second end-effector "tool" is linked to this group.

File: config/arm.xacro (robot description, xacro)
@@ -1,5 +1,5 @@
 <?xml version="1.0" encoding="UTF-8"?>
 <robot xmlns:xacro="http://www.ros.org/wiki/xacro" name="panda">
-    <xacro:macro name="arm">
+    <xacro:macro name="arm" params="name tip_link">
         <!--GROUPS: Representation of a set of joints and links. This can be useful for specifying DOF to plan for, defining arms, end effectors, etc-->
         <!--LINKS: When a link is specified, the parent joint of that link (if it exists) is automatically included-->
@@ -7,9 +7,9 @@
         <!--CHAINS: When a chain is specified, all the links along the chain (including endpoints) are included in the group. Additionally, all the joints that are parents to included links are also included. This means that joints along the chain and the parent joint of the base link are included in the group-->
         <!--SUBGROUPS: Groups can also be formed by referencing to already defined group names-->
-        <group name="panda_arm">
-            <chain base_link="panda_link0" tip_link="panda_tool" />
+        <group name="${name}">
+            <chain base_link="panda_link0" tip_link="${tip_link}" />
         </group>
         <!--GROUP STATES: Purpose: Define a named state for a particular group, in terms of joint values. This is useful to define states like 'folded arms'-->
-        <group_state name="ready" group="panda_arm">
+        <group_state name="ready" group="${name}">
             <joint name="panda_joint1" value="0" />
             <joint name="panda_joint2" value="${-pi/4}" />
@@ -20,5 +20,5 @@
             <joint name="panda_joint7" value="${pi/4}" />
         </group_state>
-        <group_state name="extended" group="panda_arm">
+        <group_state name="extended" group="${name}">
             <joint name="panda_joint1" value="0" />
             <joint name="panda_joint2" value="0" />
@@ -29,32 +29,32 @@
             <joint name="panda_joint7" value="${pi/4}" />
         </group_state>
-        <!--VIRTUAL JOINT: Purpose: this element defines a virtual joint between a robot link and an external frame of reference (considered fixed with respect to the robot)-->
-        <virtual_joint name="virtual_joint" type="fixed" parent_frame="world" child_link="panda_link0"/>
-        <!--DISABLE COLLISIONS: By default it is assumed that any link of the robot could potentially come into collision with any other link in the robot. This tag disables collision checking between a specified pair of links. -->
-        <disable_collisions link1="panda_link0" link2="panda_link1" reason="Adjacent"/>
-        <disable_collisions link1="panda_link0" link2="panda_link2" reason="Never"/>
-        <disable_collisions link1="panda_link0" link2="panda_link3" reason="Never"/>
-        <disable_collisions link1="panda_link0" link2="panda_link4" reason="Never"/>
-        <disable_collisions link1="panda_link1" link2="panda_link2" reason="Adjacent"/>
-        <disable_collisions link1="panda_link1" link2="panda_link3" reason="Default"/>
-        <disable_collisions link1="panda_link1" link2="panda_link4" reason="Never"/>
-        <disable_collisions link1="panda_link2" link2="panda_link3" reason="Adjacent"/>
-        <disable_collisions link1="panda_link2" link2="panda_link4" reason="Never"/>
-        <disable_collisions link1="panda_link3" link2="panda_link4" reason="Adjacent"/>
-        <disable_collisions link1="panda_link3" link2="panda_link5" reason="Default" />
-        <disable_collisions link1="panda_link3" link2="panda_link6" reason="Never"/>
-        <disable_collisions link1="panda_link4" link2="panda_link5" reason="Adjacent"/>
-        <disable_collisions link1="panda_link4" link2="panda_link6" reason="Never"/>
-        <disable_collisions link1="panda_link4" link2="panda_link7" reason="Never"/>
-        <disable_collisions link1="panda_link4" link2="panda_link8" reason="Never"/>
-        <disable_collisions link1="panda_link5" link2="panda_link6" reason="Adjacent"/>
-        <disable_collisions link1="panda_link5" link2="panda_link7" reason="Default"/>
-        <disable_collisions link1="panda_link6" link2="panda_link7" reason="Adjacent"/>
-        <disable_collisions link1="panda_link7" link2="panda_link8" reason="Adjacent"/>
-        <!-- Fix self-collisions between coarse collision geometries provided by franka_description
-             (see https://github.com/ros-planning/panda_moveit_config/pull/35#pullrequestreview-390715967).
-             These collisions are handled by joint limits already and thus can be disabled here. -->
-        <disable_collisions link1="panda_link5" link2="panda_link8" reason="Default"/>
-        <disable_collisions link1="panda_link6" link2="panda_link8" reason="Default"/>
     </xacro:macro>
+    <!--VIRTUAL JOINT: Purpose: this element defines a virtual joint between a robot link and an external frame of reference (considered fixed with respect to the robot)-->
+    <virtual_joint name="virtual_joint" type="fixed" parent_frame="world" child_link="panda_link0" />
+    <!--DISABLE COLLISIONS: By default it is assumed that any link of the robot could potentially come into collision with any other link in the robot. This tag disables collision checking between a specified pair of links. -->
+    <disable_collisions link1="panda_link0" link2="panda_link1" reason="Adjacent" />
+    <disable_collisions link1="panda_link0" link2="panda_link2" reason="Never" />
+    <disable_collisions link1="panda_link0" link2="panda_link3" reason="Never" />
+    <disable_collisions link1="panda_link0" link2="panda_link4" reason="Never" />
+    <disable_collisions link1="panda_link1" link2="panda_link2" reason="Adjacent" />
+    <disable_collisions link1="panda_link1" link2="panda_link3" reason="Default" />
+    <disable_collisions link1="panda_link1" link2="panda_link4" reason="Never" />
+    <disable_collisions link1="panda_link2" link2="panda_link3" reason="Adjacent" />
+    <disable_collisions link1="panda_link2" link2="panda_link4" reason="Never" />
+    <disable_collisions link1="panda_link3" link2="panda_link4" reason="Adjacent" />
+    <disable_collisions link1="panda_link3" link2="panda_link5" reason="Default" />
+    <disable_collisions link1="panda_link3" link2="panda_link6" reason="Never" />
+    <disable_collisions link1="panda_link4" link2="panda_link5" reason="Adjacent" />
+    <disable_collisions link1="panda_link4" link2="panda_link6" reason="Never" />
+    <disable_collisions link1="panda_link4" link2="panda_link7" reason="Never" />
+    <disable_collisions link1="panda_link4" link2="panda_link8" reason="Never" />
+    <disable_collisions link1="panda_link5" link2="panda_link6" reason="Adjacent" />
+    <disable_collisions link1="panda_link5" link2="panda_link7" reason="Default" />
+    <disable_collisions link1="panda_link6" link2="panda_link7" reason="Adjacent" />
+    <disable_collisions link1="panda_link7" link2="panda_link8" reason="Adjacent" />
+    <!-- Fix self-collisions between coarse collision geometries provided by franka_description
+            (see https://github.com/ros-planning/panda_moveit_config/pull/35#pullrequestreview-390715967).
+            These collisions are handled by joint limits already and thus can be disabled here. -->
+    <disable_collisions link1="panda_link5" link2="panda_link8" reason="Default" />
+    <disable_collisions link1="panda_link6" link2="panda_link8" reason="Default" />
 </robot>

File: config/panda.srdf.xacro (robot description, xacro)
@@ -6,5 +6,7 @@
 <robot xmlns:xacro="http://www.ros.org/wiki/xacro" name="panda">
     <xacro:include filename="$(find panda_moveit_config)/config/arm.xacro" />
-    <xacro:arm />
+    <xacro:arm name="arm" tip_link="panda_tool" />
+    <!-- old group name with old end-effector link -->
+    <xacro:arm name="panda_arm" tip_link="panda_link8"/>
     <xacro:arg name="hand" default="false" />
     <!--Add the hand if people request it-->
@@ -13,5 +15,7 @@
         <xacro:hand />
         <!--END EFFECTOR: Purpose: Represent information about an end effector.-->
-        <end_effector name="hand" parent_link="panda_tool" group="hand" parent_group="panda_arm" />
+        <end_effector name="tool" parent_link="panda_tool" group="hand" parent_group="arm" />
+        <!-- old end-effector -->
+        <end_effector name="hand" parent_link="panda_link8" group="hand" parent_group="panda_arm" />
     </xacro:if>
 </robot>

Commit message: Adaptions for https://github.com/frankaemika/franka_ros/pull/199

File: config/arm.xacro (robot description, xacro)
@@ -32,29 +32,49 @@
     <!--VIRTUAL JOINT: Purpose: this element defines a virtual joint between a robot link and an external frame of reference (considered fixed with respect to the robot)-->
     <virtual_joint name="virtual_joint" type="fixed" parent_frame="world" child_link="panda_link0" />
-    <!--DISABLE COLLISIONS: By default it is assumed that any link of the robot could potentially come into collision with any other link in the robot. This tag disables collision checking between a specified pair of links. -->
-    <disable_collisions link1="panda_link0" link2="panda_link1" reason="Adjacent" />
-    <disable_collisions link1="panda_link0" link2="panda_link2" reason="Never" />
-    <disable_collisions link1="panda_link0" link2="panda_link3" reason="Never" />
-    <disable_collisions link1="panda_link0" link2="panda_link4" reason="Never" />
-    <disable_collisions link1="panda_link1" link2="panda_link2" reason="Adjacent" />
-    <disable_collisions link1="panda_link1" link2="panda_link3" reason="Default" />
-    <disable_collisions link1="panda_link1" link2="panda_link4" reason="Never" />
-    <disable_collisions link1="panda_link2" link2="panda_link3" reason="Adjacent" />
-    <disable_collisions link1="panda_link2" link2="panda_link4" reason="Never" />
-    <disable_collisions link1="panda_link3" link2="panda_link4" reason="Adjacent" />
-    <disable_collisions link1="panda_link3" link2="panda_link5" reason="Default" />
-    <disable_collisions link1="panda_link3" link2="panda_link6" reason="Never" />
-    <disable_collisions link1="panda_link4" link2="panda_link5" reason="Adjacent" />
-    <disable_collisions link1="panda_link4" link2="panda_link6" reason="Never" />
-    <disable_collisions link1="panda_link4" link2="panda_link7" reason="Never" />
-    <disable_collisions link1="panda_link4" link2="panda_link8" reason="Never" />
-    <disable_collisions link1="panda_link5" link2="panda_link6" reason="Adjacent" />
-    <disable_collisions link1="panda_link5" link2="panda_link7" reason="Default" />
-    <disable_collisions link1="panda_link6" link2="panda_link7" reason="Adjacent" />
-    <disable_collisions link1="panda_link7" link2="panda_link8" reason="Adjacent" />
-    <!-- Fix self-collisions between coarse collision geometries provided by franka_description
-            (see https://github.com/ros-planning/panda_moveit_config/pull/35#pullrequestreview-390715967).
-            These collisions are handled by joint limits already and thus can be disabled here. -->
-    <disable_collisions link1="panda_link5" link2="panda_link8" reason="Default" />
-    <disable_collisions link1="panda_link6" link2="panda_link8" reason="Default" />
+    <xacro:macro name="collision" params="link">
+        <!-- Enable (environmental) collisions of ${link}_sc -->
+        <collision_default link="${link}_sc" allow="ALWAYS" />
+        <!-- Disable collisions of link with any other arm link, as these are handled by the "sc" links -->
+        <disable_collisions link1="${link}" link2="panda_link0" reason="Default" />
+        <disable_collisions link1="${link}" link2="panda_link1" reason="Default" />
+        <disable_collisions link1="${link}" link2="panda_link2" reason="Default" />
+        <disable_collisions link1="${link}" link2="panda_link3" reason="Default" />
+        <disable_collisions link1="${link}" link2="panda_link4" reason="Default" />
+        <disable_collisions link1="${link}" link2="panda_link5" reason="Default" />
+        <disable_collisions link1="${link}" link2="panda_link6" reason="Default" />
+        <disable_collisions link1="${link}" link2="panda_link7" reason="Default" />
+        <disable_collisions link1="${link}" link2="panda_link8" reason="Default" />
+        <disable_collisions link1="${link}_sc" link2="panda_link0" reason="Default" />
+        <disable_collisions link1="${link}_sc" link2="panda_link1" reason="Default" />
+        <disable_collisions link1="${link}_sc" link2="panda_link2" reason="Default" />
+        <disable_collisions link1="${link}_sc" link2="panda_link3" reason="Default" />
+        <disable_collisions link1="${link}_sc" link2="panda_link4" reason="Default" />
+        <disable_collisions link1="${link}_sc" link2="panda_link5" reason="Default" />
+        <disable_collisions link1="${link}_sc" link2="panda_link6" reason="Default" />
+        <disable_collisions link1="${link}_sc" link2="panda_link7" reason="Default" />
+        <disable_collisions link1="${link}_sc" link2="panda_link8" reason="Default" />
+    </xacro:macro>
+    <xacro:collision link="panda_link0"/>
+    <enable_collisions link1="panda_link0_sc" link2="panda_link5_sc" />
+    <enable_collisions link1="panda_link0_sc" link2="panda_link6_sc" />
+    <enable_collisions link1="panda_link0_sc" link2="panda_link7_sc" />
+    <enable_collisions link1="panda_link0_sc" link2="panda_link8_sc" />
+    <xacro:collision link="panda_link1" />
+    <enable_collisions link1="panda_link1_sc" link2="panda_link5_sc" />
+    <enable_collisions link1="panda_link1_sc" link2="panda_link6_sc" />
+    <enable_collisions link1="panda_link1_sc" link2="panda_link7_sc" />
+    <enable_collisions link1="panda_link1_sc" link2="panda_link8_sc" />
+    <xacro:collision link="panda_link2" />
+    <enable_collisions link1="panda_link2_sc" link2="panda_link5_sc" />
+    <enable_collisions link1="panda_link2_sc" link2="panda_link6_sc" />
+    <enable_collisions link1="panda_link2_sc" link2="panda_link7_sc" />
+    <enable_collisions link1="panda_link2_sc" link2="panda_link8_sc" />
+    <xacro:collision link="panda_link3" />
+    <enable_collisions link1="panda_link3_sc" link2="panda_link7_sc" />
+    <enable_collisions link1="panda_link3_sc" link2="panda_link8_sc" />
+    <xacro:collision link="panda_link4" />
+    <xacro:collision link="panda_link5" />
+    <xacro:collision link="panda_link6" />
+    <xacro:collision link="panda_link7" />
+    <xacro:collision link="panda_link8" />
 </robot>

File: config/hand.xacro (robot description, xacro)
@@ -14,5 +14,5 @@
         <disable_collisions link1="${finger}" link2="panda_link8" reason="Default" />
         <disable_collisions link1="${finger}" link2="panda_hand" reason="Default" />
-        <disable_collisions link1="${finger}" link2="panda_hand_coarse" reason="Default" />
+        <disable_collisions link1="${finger}" link2="panda_hand_sc" reason="Default" />
     </xacro:macro>
     <xacro:macro name="hand">
@@ -40,9 +40,17 @@
         <!--PASSIVE JOINT: Purpose: this element is used to mark joints that are not actuated-->
         <!--DISABLE COLLISIONS: By default it is assumed that any link of the robot could potentially come into collision with any other link in the robot. This tag disables collision checking between a specified pair of links. -->
-        <collision_default link="panda_hand_coarse" allow="ALWAYS" />
-        <enable_collisions link1="panda_hand_coarse" link2="panda_link0" />
-        <enable_collisions link1="panda_hand_coarse" link2="panda_link1" />
-        <enable_collisions link1="panda_hand_coarse" link2="panda_link2" />
-        <enable_collisions link1="panda_hand_coarse" link2="panda_link3" />
+        <collision_default link="panda_hand_sc" allow="ALWAYS" />
+        <enable_collisions link1="panda_hand_sc" link2="panda_link0" />
+        <enable_collisions link1="panda_hand_sc" link2="panda_link1" />
+        <enable_collisions link1="panda_hand_sc" link2="panda_link2" />
+        <enable_collisions link1="panda_hand_sc" link2="panda_link3" />
+        <!-- Disable collision of hand with all arm links. These are handled by the *_sc links -->
+        <disable_collisions link1="panda_hand" link2="panda_link0" />
+        <disable_collisions link1="panda_hand" link2="panda_link1" />
+        <disable_collisions link1="panda_hand" link2="panda_link2" />
+        <disable_collisions link1="panda_hand" link2="panda_link3" />
+        <disable_collisions link1="panda_hand" link2="panda_link4" />
+        <disable_collisions link1="panda_hand" link2="panda_link5" />
+        <disable_collisions link1="panda_hand" link2="panda_link6" />
         <disable_collisions link1="panda_hand" link2="panda_link7" />
         <disable_collisions link1="panda_hand" link2="panda_link8" />
