Commit message: added arm_id variable such that moveit can plan for different panda robots

File: config/arm.xacro (robot description, xacro)
@@ -8,73 +8,73 @@
         <!--SUBGROUPS: Groups can also be formed by referencing to already defined group names-->
         <group name="${name}">
-            <chain base_link="panda_link0" tip_link="${tip_link}" />
+            <chain base_link="$(arg arm_id)_link0" tip_link="${tip_link}" />
         </group>
         <!--GROUP STATES: Purpose: Define a named state for a particular group, in terms of joint values. This is useful to define states like 'folded arms'-->
         <group_state name="ready" group="${name}">
-            <joint name="panda_joint1" value="0" />
-            <joint name="panda_joint2" value="${-pi/4}" />
-            <joint name="panda_joint3" value="0" />
-            <joint name="panda_joint4" value="${-3*pi/4}" />
-            <joint name="panda_joint5" value="0" />
-            <joint name="panda_joint6" value="${pi/2}" />
-            <joint name="panda_joint7" value="${pi/4}" />
+            <joint name="$(arg arm_id)_joint1" value="0" />
+            <joint name="$(arg arm_id)_joint2" value="${-pi/4}" />
+            <joint name="$(arg arm_id)_joint3" value="0" />
+            <joint name="$(arg arm_id)_joint4" value="${-3*pi/4}" />
+            <joint name="$(arg arm_id)_joint5" value="0" />
+            <joint name="$(arg arm_id)_joint6" value="${pi/2}" />
+            <joint name="$(arg arm_id)_joint7" value="${pi/4}" />
         </group_state>
         <group_state name="extended" group="${name}">
-            <joint name="panda_joint1" value="0" />
-            <joint name="panda_joint2" value="0" />
-            <joint name="panda_joint3" value="0" />
-            <joint name="panda_joint4" value="-0.1" />
-            <joint name="panda_joint5" value="0" />
-            <joint name="panda_joint6" value="${pi}" />
-            <joint name="panda_joint7" value="${pi/4}" />
+            <joint name="$(arg arm_id)_joint1" value="0" />
+            <joint name="$(arg arm_id)_joint2" value="0" />
+            <joint name="$(arg arm_id)_joint3" value="0" />
+            <joint name="$(arg arm_id)_joint4" value="-0.1" />
+            <joint name="$(arg arm_id)_joint5" value="0" />
+            <joint name="$(arg arm_id)_joint6" value="${pi}" />
+            <joint name="$(arg arm_id)_joint7" value="${pi/4}" />
         </group_state>
     </xacro:macro>
     <!--VIRTUAL JOINT: Purpose: this element defines a virtual joint between a robot link and an external frame of reference (considered fixed with respect to the robot)-->
-    <virtual_joint name="virtual_joint" type="fixed" parent_frame="world" child_link="panda_link0" />
+    <virtual_joint name="virtual_joint" type="fixed" parent_frame="world" child_link="$(arg arm_id)_link0" />
     <xacro:macro name="collision" params="link">
         <!-- Enable (environmental) collisions of ${link}_sc -->
         <disable_default_collisions link="${link}_sc" />
         <!-- Disable collisions of link with any other arm link, as these are handled by the "sc" links -->
-        <disable_collisions link1="${link}" link2="panda_link0" reason="Default" />
-        <disable_collisions link1="${link}" link2="panda_link1" reason="Default" />
-        <disable_collisions link1="${link}" link2="panda_link2" reason="Default" />
-        <disable_collisions link1="${link}" link2="panda_link3" reason="Default" />
-        <disable_collisions link1="${link}" link2="panda_link4" reason="Default" />
-        <disable_collisions link1="${link}" link2="panda_link5" reason="Default" />
-        <disable_collisions link1="${link}" link2="panda_link6" reason="Default" />
-        <disable_collisions link1="${link}" link2="panda_link7" reason="Default" />
-        <disable_collisions link1="${link}" link2="panda_link8" reason="Default" />
-        <disable_collisions link1="${link}_sc" link2="panda_link0" reason="Default" />
-        <disable_collisions link1="${link}_sc" link2="panda_link1" reason="Default" />
-        <disable_collisions link1="${link}_sc" link2="panda_link2" reason="Default" />
-        <disable_collisions link1="${link}_sc" link2="panda_link3" reason="Default" />
-        <disable_collisions link1="${link}_sc" link2="panda_link4" reason="Default" />
-        <disable_collisions link1="${link}_sc" link2="panda_link5" reason="Default" />
-        <disable_collisions link1="${link}_sc" link2="panda_link6" reason="Default" />
-        <disable_collisions link1="${link}_sc" link2="panda_link7" reason="Default" />
-        <disable_collisions link1="${link}_sc" link2="panda_link8" reason="Default" />
+        <disable_collisions link1="${link}" link2="$(arg arm_id)_link0" reason="Default" />
+        <disable_collisions link1="${link}" link2="$(arg arm_id)_link1" reason="Default" />
+        <disable_collisions link1="${link}" link2="$(arg arm_id)_link2" reason="Default" />
+        <disable_collisions link1="${link}" link2="$(arg arm_id)_link3" reason="Default" />
+        <disable_collisions link1="${link}" link2="$(arg arm_id)_link4" reason="Default" />
+        <disable_collisions link1="${link}" link2="$(arg arm_id)_link5" reason="Default" />
+        <disable_collisions link1="${link}" link2="$(arg arm_id)_link6" reason="Default" />
+        <disable_collisions link1="${link}" link2="$(arg arm_id)_link7" reason="Default" />
+        <disable_collisions link1="${link}" link2="$(arg arm_id)_link8" reason="Default" />
+        <disable_collisions link1="${link}_sc" link2="$(arg arm_id)_link0" reason="Default" />
+        <disable_collisions link1="${link}_sc" link2="$(arg arm_id)_link1" reason="Default" />
+        <disable_collisions link1="${link}_sc" link2="$(arg arm_id)_link2" reason="Default" />
+        <disable_collisions link1="${link}_sc" link2="$(arg arm_id)_link3" reason="Default" />
+        <disable_collisions link1="${link}_sc" link2="$(arg arm_id)_link4" reason="Default" />
+        <disable_collisions link1="${link}_sc" link2="$(arg arm_id)_link5" reason="Default" />
+        <disable_collisions link1="${link}_sc" link2="$(arg arm_id)_link6" reason="Default" />
+        <disable_collisions link1="${link}_sc" link2="$(arg arm_id)_link7" reason="Default" />
+        <disable_collisions link1="${link}_sc" link2="$(arg arm_id)_link8" reason="Default" />
     </xacro:macro>
-    <xacro:collision link="panda_link0"/>
-    <enable_collisions link1="panda_link0_sc" link2="panda_link5_sc" />
-    <enable_collisions link1="panda_link0_sc" link2="panda_link6_sc" />
-    <enable_collisions link1="panda_link0_sc" link2="panda_link7_sc" />
-    <enable_collisions link1="panda_link0_sc" link2="panda_link8_sc" />
-    <xacro:collision link="panda_link1" />
-    <enable_collisions link1="panda_link1_sc" link2="panda_link5_sc" />
-    <enable_collisions link1="panda_link1_sc" link2="panda_link6_sc" />
-    <enable_collisions link1="panda_link1_sc" link2="panda_link7_sc" />
-    <enable_collisions link1="panda_link1_sc" link2="panda_link8_sc" />
-    <xacro:collision link="panda_link2" />
-    <enable_collisions link1="panda_link2_sc" link2="panda_link5_sc" />
-    <enable_collisions link1="panda_link2_sc" link2="panda_link6_sc" />
-    <enable_collisions link1="panda_link2_sc" link2="panda_link7_sc" />
-    <enable_collisions link1="panda_link2_sc" link2="panda_link8_sc" />
-    <xacro:collision link="panda_link3" />
-    <enable_collisions link1="panda_link3_sc" link2="panda_link7_sc" />
-    <enable_collisions link1="panda_link3_sc" link2="panda_link8_sc" />
-    <xacro:collision link="panda_link4" />
-    <xacro:collision link="panda_link5" />
-    <xacro:collision link="panda_link6" />
-    <xacro:collision link="panda_link7" />
-    <xacro:collision link="panda_link8" />
+    <xacro:collision link="$(arg arm_id)_link0"/>
+    <enable_collisions link1="$(arg arm_id)_link0_sc" link2="$(arg arm_id)_link5_sc" />
+    <enable_collisions link1="$(arg arm_id)_link0_sc" link2="$(arg arm_id)_link6_sc" />
+    <enable_collisions link1="$(arg arm_id)_link0_sc" link2="$(arg arm_id)_link7_sc" />
+    <enable_collisions link1="$(arg arm_id)_link0_sc" link2="$(arg arm_id)_link8_sc" />
+    <xacro:collision link="$(arg arm_id)_link1" />
+    <enable_collisions link1="$(arg arm_id)_link1_sc" link2="$(arg arm_id)_link5_sc" />
+    <enable_collisions link1="$(arg arm_id)_link1_sc" link2="$(arg arm_id)_link6_sc" />
+    <enable_collisions link1="$(arg arm_id)_link1_sc" link2="$(arg arm_id)_link7_sc" />
+    <enable_collisions link1="$(arg arm_id)_link1_sc" link2="$(arg arm_id)_link8_sc" />
+    <xacro:collision link="$(arg arm_id)_link2" />
+    <enable_collisions link1="$(arg arm_id)_link2_sc" link2="$(arg arm_id)_link5_sc" />
+    <enable_collisions link1="$(arg arm_id)_link2_sc" link2="$(arg arm_id)_link6_sc" />
+    <enable_collisions link1="$(arg arm_id)_link2_sc" link2="$(arg arm_id)_link7_sc" />
+    <enable_collisions link1="$(arg arm_id)_link2_sc" link2="$(arg arm_id)_link8_sc" />
+    <xacro:collision link="$(arg arm_id)_link3" />
+    <enable_collisions link1="$(arg arm_id)_link3_sc" link2="$(arg arm_id)_link7_sc" />
+    <enable_collisions link1="$(arg arm_id)_link3_sc" link2="$(arg arm_id)_link8_sc" />
+    <xacro:collision link="$(arg arm_id)_link4" />
+    <xacro:collision link="$(arg arm_id)_link5" />
+    <xacro:collision link="$(arg arm_id)_link6" />
+    <xacro:collision link="$(arg arm_id)_link7" />
+    <xacro:collision link="$(arg arm_id)_link8" />
 </robot>

File: config/hand.xacro (robot description, xacro)
@@ -4,15 +4,15 @@
         <!-- Disable all self-collisions between finger and arm links,
              as these are already covered by the coarser hand collision model -->
-        <disable_collisions link1="${finger}" link2="panda_link0" reason="Default" />
-        <disable_collisions link1="${finger}" link2="panda_link1" reason="Default" />
-        <disable_collisions link1="${finger}" link2="panda_link2" reason="Default" />
-        <disable_collisions link1="${finger}" link2="panda_link3" reason="Default" />
-        <disable_collisions link1="${finger}" link2="panda_link4" reason="Default" />
-        <disable_collisions link1="${finger}" link2="panda_link5" reason="Default" />
-        <disable_collisions link1="${finger}" link2="panda_link6" reason="Default" />
-        <disable_collisions link1="${finger}" link2="panda_link7" reason="Default" />
-        <disable_collisions link1="${finger}" link2="panda_link8" reason="Default" />
-        <disable_collisions link1="${finger}" link2="panda_hand" reason="Default" />
-        <disable_collisions link1="${finger}" link2="panda_hand_sc" reason="Default" />
+        <disable_collisions link1="${finger}" link2="$(arg arm_id)_link0" reason="Default" />
+        <disable_collisions link1="${finger}" link2="$(arg arm_id)_link1" reason="Default" />
+        <disable_collisions link1="${finger}" link2="$(arg arm_id)_link2" reason="Default" />
+        <disable_collisions link1="${finger}" link2="$(arg arm_id)_link3" reason="Default" />
+        <disable_collisions link1="${finger}" link2="$(arg arm_id)_link4" reason="Default" />
+        <disable_collisions link1="${finger}" link2="$(arg arm_id)_link5" reason="Default" />
+        <disable_collisions link1="${finger}" link2="$(arg arm_id)_link6" reason="Default" />
+        <disable_collisions link1="${finger}" link2="$(arg arm_id)_link7" reason="Default" />
+        <disable_collisions link1="${finger}" link2="$(arg arm_id)_link8" reason="Default" />
+        <disable_collisions link1="${finger}" link2="$(arg arm_id)_hand" reason="Default" />
+        <disable_collisions link1="${finger}" link2="$(arg arm_id)_hand_sc" reason="Default" />
     </xacro:macro>
     <xacro:macro name="hand">
@@ -23,16 +23,16 @@
         <!--SUBGROUPS: Groups can also be formed by referencing to already defined group names-->
         <group name="hand">
-            <link name="panda_hand"/>
-            <link name="panda_leftfinger"/>
-            <link name="panda_rightfinger"/>
+            <link name="$(arg arm_id)_hand"/>
+            <link name="$(arg arm_id)_leftfinger"/>
+            <link name="$(arg arm_id)_rightfinger"/>
         </group>
         <!--GROUP STATES: Purpose: Define a named state for a particular group, in terms of joint values. This is useful to define states like 'folded arms'-->
         <group_state name="open" group="hand">
-            <joint name="panda_finger_joint1" value="0.035"/>
-            <joint name="panda_finger_joint2" value="0.035"/>
+            <joint name="$(arg arm_id)_finger_joint1" value="0.035"/>
+            <joint name="$(arg arm_id)_finger_joint2" value="0.035"/>
         </group_state>
         <group_state name="close" group="hand">
-            <joint name="panda_finger_joint1" value="0"/>
-            <joint name="panda_finger_joint2" value="0"/>
+            <joint name="$(arg arm_id)_finger_joint1" value="0"/>
+            <joint name="$(arg arm_id)_finger_joint2" value="0"/>
         </group_state>
         <!--END EFFECTOR: Purpose: Represent information about an end effector.-->
@@ -40,22 +40,22 @@
         <!--PASSIVE JOINT: Purpose: this element is used to mark joints that are not actuated-->
         <!--DISABLE COLLISIONS: By default it is assumed that any link of the robot could potentially come into collision with any other link in the robot. This tag disables collision checking between a specified pair of links. -->
-        <disable_default_collisions link="panda_hand_sc" />
-        <enable_collisions link1="panda_hand_sc" link2="panda_link0" />
-        <enable_collisions link1="panda_hand_sc" link2="panda_link1" />
-        <enable_collisions link1="panda_hand_sc" link2="panda_link2" />
-        <enable_collisions link1="panda_hand_sc" link2="panda_link3" />
+        <disable_default_collisions link="$(arg arm_id)_hand_sc" />
+        <enable_collisions link1="$(arg arm_id)_hand_sc" link2="$(arg arm_id)_link0" />
+        <enable_collisions link1="$(arg arm_id)_hand_sc" link2="$(arg arm_id)_link1" />
+        <enable_collisions link1="$(arg arm_id)_hand_sc" link2="$(arg arm_id)_link2" />
+        <enable_collisions link1="$(arg arm_id)_hand_sc" link2="$(arg arm_id)_link3" />
         <!-- Disable collision of hand with all arm links. These are handled by the *_sc links -->
-        <disable_collisions link1="panda_hand" link2="panda_link0" />
-        <disable_collisions link1="panda_hand" link2="panda_link1" />
-        <disable_collisions link1="panda_hand" link2="panda_link2" />
-        <disable_collisions link1="panda_hand" link2="panda_link3" />
-        <disable_collisions link1="panda_hand" link2="panda_link4" />
-        <disable_collisions link1="panda_hand" link2="panda_link5" />
-        <disable_collisions link1="panda_hand" link2="panda_link6" />
-        <disable_collisions link1="panda_hand" link2="panda_link7" />
-        <disable_collisions link1="panda_hand" link2="panda_link8" />
-        <xacro:finger_collisions finger="panda_leftfinger" />
-        <xacro:finger_collisions finger="panda_rightfinger" />
-        <disable_collisions link1="panda_leftfinger" link2="panda_rightfinger" reason="Default" />
+        <disable_collisions link1="$(arg arm_id)_hand" link2="$(arg arm_id)_link0" />
+        <disable_collisions link1="$(arg arm_id)_hand" link2="$(arg arm_id)_link1" />
+        <disable_collisions link1="$(arg arm_id)_hand" link2="$(arg arm_id)_link2" />
+        <disable_collisions link1="$(arg arm_id)_hand" link2="$(arg arm_id)_link3" />
+        <disable_collisions link1="$(arg arm_id)_hand" link2="$(arg arm_id)_link4" />
+        <disable_collisions link1="$(arg arm_id)_hand" link2="$(arg arm_id)_link5" />
+        <disable_collisions link1="$(arg arm_id)_hand" link2="$(arg arm_id)_link6" />
+        <disable_collisions link1="$(arg arm_id)_hand" link2="$(arg arm_id)_link7" />
+        <disable_collisions link1="$(arg arm_id)_hand" link2="$(arg arm_id)_link8" />
+        <xacro:finger_collisions finger="$(arg arm_id)_leftfinger" />
+        <xacro:finger_collisions finger="$(arg arm_id)_rightfinger" />
+        <disable_collisions link1="$(arg arm_id)_leftfinger" link2="$(arg arm_id)_rightfinger" reason="Default" />
     </xacro:macro>
 </robot>

File: config/panda.srdf.xacro (robot description, xacro)
@@ -6,7 +6,8 @@
 <robot xmlns:xacro="http://www.ros.org/wiki/xacro" name="panda">
     <xacro:include filename="$(find panda_moveit_config)/config/arm.xacro" />
-    <xacro:arm name="manipulator" tip_link="panda_hand_tcp" />
+    <xacro:arg name="arm_id" default="panda" />
+    <!-- <xacro:arm name="$(arg arm_id)_manipulator" tip_link="$(arg arm_id)_hand_tcp" arm_id="$(arg arm_id)"/> -->
     <!-- old group name with old end-effector link -->
-    <xacro:arm name="panda_arm" tip_link="panda_link8"/>
+    <xacro:arm name="$(arg arm_id)_arm" tip_link="$(arg arm_id)_link8"/>
     <xacro:arg name="hand" default="false" />
     <!--Add the hand if people request it-->
@@ -15,7 +16,7 @@
         <xacro:hand />
         <!--END EFFECTOR: Purpose: Represent information about an end effector.-->
-        <end_effector name="hand_tcp" parent_link="panda_hand_tcp" group="hand" parent_group="manipulator" />
+        <!-- <end_effector name="$(arg arm_id)_hand_tcp" parent_link="$(arg arm_id)_hand_tcp" group="hand" parent_group="$(arg arm_id)_manipulator" /> -->
         <!-- old end-effector -->
-        <end_effector name="hand" parent_link="panda_link8" group="hand" parent_group="panda_arm" />
+        <end_effector name="$(arg arm_id)_hand" parent_link="$(arg arm_id)_link8" group="hand" parent_group="$(arg arm_id)_arm" />
     </xacro:if>
 </robot>
